File: Power delivery/Schematic/Versions2/Versions3.kicad_pcb (KiCad board)
At the start: 2 copper layers, 43.2 x 33 mm, 12 parts, among them U1 TPS62932

Commit message: done
Other:
- board text added: "+24V"
- board text added: "GND"
- board text added: "V out"
Changed lines of the file:
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@@
     (property "ki_keywords" "connector")
     (attr exclude_from_pos_files)
-    (fp_text reference "Jout1" (at 1.8 -2 90) (layer "F.SilkS")
+    (fp_text reference "Jout1" (at 5.178 3.043 -180) (layer "F.SilkS")
         (effects (font (size 1 1) (thickness 0.15)))
     )
@@
     (property "ki_keywords" "connector")
     (attr exclude_from_pos_files)
-    (fp_text reference "Jin1" (at 1.8 -2 90) (layer "F.SilkS")
+    (fp_text reference "Jin1" (at -1.518 2.273 -180) (layer "F.SilkS")
         (effects (font (size 1 1) (thickness 0.15)))
     )
@@
   (gr_line (start 129.54 66.04) (end 86.36 66.04)
     (stroke (width 0.1) (type default)) (layer "Edge.Cuts"))
+  (gr_text "V out" (at 95.504 35.306) (layer "F.SilkS")
+    (effects (font (size 1 1) (thickness 0.15)) (justify left bottom))
+  )
   (gr_text "ALSET INNOVATIONS" (at 89.5 40.5 -90) (layer "F.SilkS")
     (effects (font (face "TESLA") (size 1 1) (thickness 0.15)) (justify left bottom))
@@
     )
   )
+  (gr_text "+24V" (at 95.758 61.214) (layer "F.SilkS")
+    (effects (font (size 1 1) (thickness 0.15)) (justify left bottom))
+  )
+  (gr_text "GND" (at 95.758 64.77) (layer "F.SilkS")
+    (effects (font (size 1 1) (thickness 0.15)) (justify left bottom))
+  )
+  (gr_text "GND" (at 95.25 39.116) (layer "F.SilkS")
+    (effects (font (size 1 1) (thickness 0.15)) (justify left bottom))
+  )
   (segment (start 123.453 58.547) (end 125 57) (width 0.25) (layer "F.Cu") (net 1))
