File: Version 1/Version 1_test2.kicad_pcb (KiCad board)
At the start: 2 copper layers, 97.2 x 106 mm, 83 parts, among them J1 Conn_01x05, Q1 IPP015N04NF2SAKMA1, Q2 IPP015N04NF2SAKMA1, Q3 IPP015N04NF2SAKMA1, Q4 IPP015N04NF2SAKMA1, Q5 IPP015N04NF2SAKMA1, Q6 IPP015N04NF2SAKMA1, U1 TPS62932, U2 TPS62932, U3 TPS62932, U4 IRS2004, U5 IRS2004, U6 IRS2004, U7 YAAJ_BlackPill_SWD_BreakoutV2, U8 ACS712xLCTR-05B

Commit message: updated SCHEMATIC
Parts:
- removed U8: ACS712xLCTR-05B, Package_SO:SOIC-8_3.9x4.9mm_P1.27mm
- added Cbypass-ACS37002: C, Capacitor_THT:C_Disc_D3.4mm_W2.1mm_P2.50mm, F.Cu at (94.9, 100.2)
- added Cl-ACS37002: C, Capacitor_THT:C_Disc_D3.4mm_W2.1mm_P2.50mm, F.Cu at (94.9, 103.8)
- added Cref-ACS37002: C, Capacitor_THT:C_Disc_D3.4mm_W2.1mm_P2.50mm, F.Cu at (94.9, 107.5)
- added Cvoc-ACS37002: C, Capacitor_THT:C_Disc_D3.4mm_W2.1mm_P2.50mm, F.Cu at (94.9, 111.1)
- added IC1: ACS37002LLAATR-015B5, KiCad:SOIC127P1030X265-16N, F.Cu at (83.1, 103.4)
- added Rvoch-ACS37002: R, Resistor_THT:R_Axial_DIN0207_L6.3mm_D2.5mm_P10.16mm_Horizontal, F.Cu at (107.1, 114.2)
- added Rvocl-ACS37002: R, Resistor_THT:R_Axial_DIN0207_L6.3mm_D2.5mm_P10.16mm_Horizontal, F.Cu at (103.4, 114.2)
